Commit message: 区域赛版本

File: rm_vision/rm_gimbal_description-main/rm_gimbal_description-main/urdf/rm_gimbal.urdf.xacro (robot description, xacro)
@@ -1,26 +1,28 @@
 <?xml version="1.0" encoding="utf-8"?>
-<robot name="rm_gimbal"
-  xmlns:xacro="http://ros.org/wiki/xacro">
-  <xacro:arg name="xyz" default="0 0 0.05" />
+<robot name="rm_gimbal" xmlns:xacro="http://ros.org/wiki/xacro">
+  <xacro:arg name="odom2gimbal" default="0 0 0" />
+  <xacro:arg name="giambal2camera" default="0.08 0 0.063 " />
+  <!-- <xacro:arg name="giambal2camera" default="0.1 -0.06 0.00 " /> -->
   <xacro:arg name="rpy" default="0 0 0" />
   <link name="odom" />
-  <link name="gimbal_link" />
-  <joint name="gimbal_joint" type="floating">
-    <origin xyz="$(arg xyz)" rpy="0 0 0" />
+  <joint name="gimbal_joint" type="fixed">
+    <origin xyz="$(arg odom2gimbal)" rpy="0 0 0" />
     <parent link="odom" />
     <child link="gimbal_link" />
   </joint>
-  <link name="camera_link" />
+  <link name="gimbal_link" />
   <joint name="camera_joint" type="fixed">
-    <origin xyz="$(arg xyz)" rpy="$(arg rpy) "/>
+    <origin xyz="$(arg giambal2camera)" rpy="$(arg rpy) "/>
     <parent link="gimbal_link" />
     <child link="camera_link" />
     <axis xyz="0 0 0" />
   </joint>
-  <link name="camera_optical_frame" />
+  <link name="camera_link" />
   <joint name="camera_optical_joint" type="fixed">
+    <!-- <origin xyz="0 0 0" rpy="-1.579522 0 ${-pi/2}" /> -->
     <origin xyz="0 0 0" rpy="${-pi/2} 0 ${-pi/2}" />
     <parent link="camera_link" />
     <child link="camera_optical_frame" />
   </joint>
+  <link name="camera_optical_frame" />
 </robot>

Commit message: 最新改进

File: rm_vision/rm_gimbal_description-main/rm_gimbal_description-main/urdf/rm_gimbal.urdf.xacro (robot description, xacro)
@@ -20,6 +20,6 @@
   <link name="camera_link" />
   <joint name="camera_optical_joint" type="fixed">
-    <!-- <origin xyz="0 0 0" rpy="-1.579522 0 ${-pi/2}" /> -->
-    <origin xyz="0 0 0" rpy="${-pi/2} 0 ${-pi/2}" />
+    <origin xyz="0 0 0" rpy="-1.589522 0 ${-pi/2}" />
+    <!-- <origin xyz="0 0 0" rpy="${-pi/2} 0 ${-pi/2}" /> -->
     <parent link="camera_link" />
     <child link="camera_optical_frame" />
